Commit message: Created robot control and environmet

File: description/robot_core.xacro (robot description, xacro)
@@ -41,4 +41,7 @@
         </xacro:inertial_cylinder>
     </link>
+    <gazebo reference="chassis">
+        <material>Gazebo/Orange</material>
+    </gazebo>
     <!-- LEFT WHEEL LINK-->
     <joint name= "left_wheel_joint" type="continuous">
@@ -64,4 +67,7 @@
         </xacro:inertial_cylinder>
     </link>
+    <gazebo reference="left_wheel">
+        <material>Gazebo/Black</material>
+    </gazebo>
     <!-- RIGHT WHEEL LINK-->
     <joint name= "right_wheel_joint" type="continuous">
@@ -87,5 +93,8 @@
         </xacro:inertial_cylinder>
     </link>
-    <!-- CASTER WHEEL FRONT-->
+    <gazebo reference="right_wheel">
+        <material>Gazebo/Black</material>
+    </gazebo>
+    <!-- CASTER FRONT WHEEL-->
     <joint name="caster_wheel_front_joint" type="fixed">
         <parent link="chassis"/>
@@ -109,5 +118,10 @@
         </xacro:inertial_sphere>
     </link>
-    <!-- CASTER WHEEL BACK-->
+    <gazebo reference="caster_wheel_front">
+        <material>Gazebo/White</material>
+        <mu1 value="0.001"/>
+        <mu2 value="0.001"/>
+    </gazebo>
+    <!-- CASTER BACK WHEEL-->
     <joint name="caster_wheel_back_joint" type="fixed">
         <parent link="chassis"/>
@@ -131,3 +145,8 @@
         </xacro:inertial_sphere>
     </link>
+    <gazebo reference="caster_wheel_back">
+        <material>Gazebo/White</material>
+        <mu1 value="0.001"/>
+        <mu2 value="0.001"/>
+    </gazebo>
 </robot>

Commit message: Robot functional including odometry fusion with imu MPU6050

File: description/robot_core.xacro (robot description, xacro)
@@ -150,3 +150,29 @@
         <mu2 value="0.001"/>
     </gazebo>
+    <!-- IMU SENSOR -->
+    <joint name= "imu_sensor_joint" type="fixed">
+        <parent link="base_link"/>
+        <child link="imu_sensor"/>
+        <origin xyz="-0.07 0 0.02"/>
+    </joint>
+    <link name="imu_sensor">
+        <visual>
+            <geometry>
+                <box size="0.02 0.02 0.005"/>
+            </geometry>
+            <material name="blue"/>
+        </visual>
+        <sensor type="imu" name="imu_sensor">
+            <origin xyz="0 0 0"/>
+            <update_rate>100</update_rate>
+            <imu>
+                <angular_velocity>true</angular_velocity>
+                <linear_acceleration>true</linear_acceleration>
+                <orientation>true</orientation>
+            </imu>
+        </sensor>
+    </link>
+    <gazebo reference="chassis">
+        <material>Gazebo/Blue</material>
+    </gazebo>
 </robot>

File: description/ros2_control.xacro (robot description, xacro)
@@ -6,15 +6,15 @@
             <param name="left_wheel_name">left_wheel_joint</param>
             <param name="right_wheel_name">right_wheel_joint</param>
-            <param name="loop_rate">3</param>
+            <param name="loop_rate">5</param>
             <param name="device">/dev/ttyACM0</param>
             <param name="baud_rate">57600</param>
             <param name="timeout">1000</param>
-            <param name="left_enc_counts_per_rev">188</param>
-            <param name="right_enc_counts_per_rev">25</param>
+            <param name="left_enc_counts_per_rev">20</param>
+            <param name="right_enc_counts_per_rev">20</param>
         </hardware>
         <joint name="left_wheel_joint">
             <command_interface name="velocity">
-                <param name="min">-10</param>
-                <param name="max">10</param>
+                <param name="min">-50</param>
+                <param name="max">50</param>
             </command_interface>
             <state_interface name="velocity"/>
@@ -23,10 +23,31 @@
         <joint name="right_wheel_joint">
             <command_interface name="velocity">
-                <param name="min">-10</param>
-                <param name="max">10</param>
+                <param name="min">-50</param>
+                <param name="max">50</param>
             </command_interface>
             <state_interface name="velocity"/>
             <state_interface name="position"/>
         </joint>
+    </ros2_control>
+    <ros2_control name="ImuSensor" type="sensor">
+        <hardware>
+            <plugin>diffdrive_arduino/ImuSensorHardware</plugin>
+            <param name="imu_sensor_name">imu_sensor</param>
+            <param name="device">/dev/ttyACM0</param>
+            <param name="baud_rate">57600</param>
+            <param name="timeout">1000</param>
+        </hardware>
+        <sensor name="imu_sensor">
+            <state_interface name="orientation.x"/>
+            <state_interface name="orientation.y"/>
+            <state_interface name="orientation.z"/>
+            <state_interface name="orientation.w"/>
+            <state_interface name="angular_velocity.x"/>
+            <state_interface name="angular_velocity.y"/>
+            <state_interface name="angular_velocity.z"/>
+            <state_interface name="linear_acceleration.x"/>
+            <state_interface name="linear_acceleration.y"/>
+            <state_interface name="linear_acceleration.z"/>
+        </sensor>
     </ros2_control>
     <!-- <ros2_control name="GazeboSystem" type="system">
